File: Indira_Setu_pcb/Indira_Setu/Indira_Setu.kicad_sch (KiCad schematic)
At the start: 2 parts, among them U1 Pico

Commit message: Add files via upload
Parts:
- added U2: CR2013-MI2120, Display:CR2013-MI2120, symbol Driver_Display:CR2013-MI2120
Connections:
- net at U1.13 (GND): now also CJMCU_FT1.GND1 (GND)
- net at U1.14 (GPIO10): now also U2.7 (SCK)
- net at U1.15 (GPIO11): now also U2.6 (MOSI)
- net at U1.20 (GPIO15): now also U2.9 (MISO)
- net at U1.21 (GPIO16): now also U2.5 (D/~{C})
- net at U1.22 (GPIO17): now also U2.4 (RESET)
- net at U1.24 (GPIO18): now also U2.3 (~{CS})
- net at U1.36 (3V3): now also CJMCU_FT1.+3.3V, U2.1 (VCC), U2.8 (LED)
- net at U1.38 (GND): now also U2.2 (GND)
- now unconnected: CJMCU_FT1.GND2 (GND), U1.3 (GND), U1.8 (GND)
- no-connect marks 10 -> 27

Commit message: Add files via upload
Parts:
- added U3, U4: Pico, Indira_Setu:RPi_Pico_SMD_TH, symbol MCU_RaspberryPi_and_Boards:Pico
Connections:
- net at U1.12 (GPIO9): now also U3.7 (GPIO5), U4.7 (GPIO5)
- net at U1.3 (GND): now also U3.18 (GND)
- net at CJMCU_FT1.AC5, U1.4 (GPIO2): now also U3.4 (GPIO2), U4.4 (GPIO2)
- net at CJMCU_FT1.AC0, U1.5 (GPIO3): now also U3.5 (GPIO3), U4.5 (GPIO3)
- net at CJMCU_FT1.AC1, U1.6 (GPIO4): now also U3.6 (GPIO4), U4.6 (GPIO4)
- net at CJMCU_FT1.AD1: now also U3.9 (GPIO6)
- net at CJMCU_FT1.AD2: now also U4.9 (GPIO6)
- no-connect marks 27 -> 48
Other:
- moved on the sheet: U1, U2
